File: kicad/EricOnboardingProject/EricOnboardingProject.kicad_pcb (KiCad board)
At the start: 4 copper layers, 0 parts

Commit message: Finalized KiCad schematic, set up the PCB editor
Parts:
- added C1: 100μf, Capacitor_THT:CP_Radial_D6.3mm_P2.50mm, F.Cu at (131.7, 95.4)
- added CO1: 330μf, Diode_THT:D_DO-41_SOD81_P10.16mm_Horizontal, F.Cu at (116.9, 93.6)
- added CT1: 1500pf, Capacitor_THT:C_Disc_D5.0mm_W2.5mm_P5.00mm, F.Cu at (116.6, 118.2)
- added D1: 1N5819, Diode_THT:D_DO-41_SOD81_P10.16mm_Horizontal, F.Cu at (116.9, 97.9)
- added L1: 220 uH, Inductor_THT:L_Radial_D7.5mm_P5.00mm_Fastron_07P, F.Cu at (130.7, 116.6)
- added R1: 82Ω, Resistor_THT:R_Axial_DIN0207_L6.3mm_D2.5mm_P10.16mm_Horizontal, F.Cu at (116.6, 102.0)
- added R2: 1500Ω, Resistor_THT:R_Axial_DIN0207_L6.3mm_D2.5mm_P10.16mm_Horizontal, F.Cu at (116.6, 106.1)
- added R8: 180Ω, Resistor_THT:R_Axial_DIN0207_L6.3mm_D2.5mm_P10.16mm_Horizontal, F.Cu at (116.6, 110.1)
- added RSC1: .22Ω, Resistor_THT:R_Axial_DIN0207_L6.3mm_D2.5mm_P10.16mm_Horizontal, F.Cu at (116.6, 114.2)
- added U1: MC34063AP, Package_DIP:DIP-8_W7.62mm, F.Cu at (129.9, 102.0)
Other:
- board outline added: 50 x 70 mm
