File: kicad/EricOnboardingProject/OnboardingCircuitOverlapped.kicad_pcb (KiCad board)
At the start: 4 copper layers, 50 x 70 mm, 10 parts, among them U1 MC34063AP

Commit message: Completed the KiCad diagram!
Routing:
- net GND: track 58.4 -> 41.4 mm
